Commit message: (실패) 차량 색깔 바꾸고, 바퀴 수직으로 달았는데 바퀴가 안보임...

File: src/ds_car_description/urdf/ds_car.urdf.xacro (robot description, xacro)
@@ -1,4 +1,11 @@
 <?xml version="1.0"?>
 <robot name="ds_car" xmlns:xacro="http://www.ros.org/wiki/xacro">
+  <!-- 색상 정의 -->
+  <material name="light_blue">
+    <color rgba="0.3 0.6 1.0 1.0"/>  <!-- 밝은 파란색 -->
+  </material>
+  <material name="dark_red">
+    <color rgba="0.8 0.1 0.1 1.0"/>  <!-- 진한 빨간색 -->
+  </material>
   <!-- 차체 (Chassis) -->
   <link name="base_link">
@@ -7,5 +14,5 @@
         <box size="1.5 1.0 0.5"/>  <!-- 크기: x=1.5m, y=1.0m, z=0.5m -->
       </geometry>
-      <material name="gray"/>
+      <material name="light_blue"/>  <!-- 색상 적용 -->
     </visual>
   </link>

File: src/ds_car_description/urdf/wheel.xacro (robot description, xacro)
@@ -7,13 +7,13 @@
           <cylinder length="0.1" radius="0.2"/>  <!-- 바퀴 크기 -->
         </geometry>
-        <material name="black"/>
+        <material name="dark_red"/>  <!-- 바퀴 색상 변경 -->
       </visual>
     </link>
-    <!-- 바퀴를 차체와 연결 -->
+    <!-- 바퀴를 차체와 수직으로 연결 -->
     <joint name="${name}_joint" type="continuous">
       <parent link="${parent}"/>
       <child link="${name}"/>
-      <origin xyz="${x_pos} ${y_pos} -0.2"/>  <!-- 바퀴 위치 조정 -->
-      <axis xyz="0 1 0"/>
+      <origin xyz="${x_pos} ${y_pos} -0.2" rpy="1.57 0 0"/>  <!-- 바퀴를 수직으로 회전 -->
+      <axis xyz="0 0 1"/>  <!-- z축 기준으로 회전 -->
     </joint>
   </xacro:macro>
